Commit message: Default to shaping.gamma=1 and n-step 3, keep URDF links off the table, add report template
Co-Authored-By: Claude Opus 5.5 <noreply@anthropic.com>
Claude-Session: https://claude.ai/code/session_015TYQ7yFwJVyj4JHpfsyt3c

File: rl_grasp_sim/assets/urdf/ur5_rg2.urdf (robot description, URDF)
Before this commit: robot ur5_rg2, 13 links, 12 joints
Links:
- link base_link: geometry collision cylinder length=0.058 radius=0.075; visual cylinder length=0.058 radius=0.075
- link link_1: geometry collision cylinder length=0.026748 radius=0.06; visual cylinder length=0.026748 radius=0.06
